Commit message: many changes, does not compile

File: sim_vehicle/sensors/sensors.urdf.xacro (robot description, xacro)
@@ -1,8 +1,8 @@
 <?xml version="1.0"?>
 <robot xmlns:xacro="http://www.ros.org/wiki/xacro">
-    <xacro:macro name="gazebo_INS_devices">
+    <xacro:macro name="model2gazebo">
         <gazebo>
-            <plugin filename="libgazebo_INS_devices.so" name="gazebo_INS_devices">
-                <node_name>gazebo_ins_devices</node_name>
+            <plugin filename="libmodel2gazebo.so" name="model2gazebo">
+                <node_name>model2gazebo</node_name>
                 <rate>100</rate>
             </plugin>

File: sim_vehicle/urdf/physics.urdf.xacro (robot description, xacro)
@@ -1,25 +1,31 @@
 <?xml version="1.0"?>
 <robot name="vehicle" xmlns:xacro="http://www.ros.org/wiki/xacro">
-  <xacro:macro name="vehicle_physics" params="name">
-    <!-- BASE_LINK -->
-    <link name="base_link">
-      <inertial>
-        <mass value="208.0" />
-        <origin xyz="0 0 0" />
-        <inertia  ixx="1.391" ixy="0.004"  ixz="0.0"  iyy="6.853"  iyz="0.0"  izz="93.0" />
-      </inertial>
-      <visual>
-        <origin xyz="0.8 0 -0.2" rpy="0 0 0" />
-          <geometry>
-            <mesh filename="package://sim_vehicle/meshes/vehicle.dae"/>
-          </geometry>
-      </visual>
-      <collision>
-        <origin xyz="0 0 0.5" rpy="0 0 0"/>
-        <geometry>
-          <box size="1 1 1" />
-        </geometry>
-      </collision>
-    </link>
-  </xacro:macro>
+	<xacro:macro name="vehicle_physics" params="name">
+		<!-- BASE_LINK -->
+		<link name="base_link">
+			<inertial>
+				<mass value="10.0" />
+				<origin xyz="0 0 0" />
+				<inertia ixx="1" ixy="0" ixz="0.0" iyy="1" iyz="0.0" izz="1" />
+			</inertial>
+			<visual>
+				<origin xyz="0 0 0" rpy="0 0 0" />
+				<geometry>
+					<mesh filename="package://sim_vehicle/meshes/vehicle.dae" />
+				</geometry>
+			</visual>
+			<collision>
+				<origin xyz="0 0 0.5" rpy="0 0 0" />
+				<geometry>
+					<box size="1 1 1" />
+				</geometry>
+			</collision>
+			<gazebo>
+				<plugin filename="libmodel2gazebo.so" name="model2gazebo">
+					<node_name>model2gazebo</node_name>
+					<rate>100</rate>
+				</plugin>
+			</gazebo>
+		</link>
+	</xacro:macro>
 </robot>

File: sim_vehicle/urdf/vehicle.urdf.xacro (robot description, xacro)
@@ -10,4 +10,3 @@
     <!--  MAIN SENSORS   -->
     <!-- *************** -->
-    <xacro:gazebo_INS_devices />
 </robot>

Commit message: problems 1

File: sim_vehicle/sensors/sensors.urdf.xacro (robot description, xacro)
@@ -1,11 +1,3 @@
 <?xml version="1.0"?>
 <robot xmlns:xacro="http://www.ros.org/wiki/xacro">
-    <xacro:macro name="model2gazebo">
-        <gazebo>
-            <plugin filename="libmodel2gazebo.so" name="model2gazebo">
-                <node_name>model2gazebo</node_name>
-                <rate>100</rate>
-            </plugin>
-        </gazebo>
-    </xacro:macro>
 </robot>

File: sim_vehicle/urdf/vehicle.urdf.xacro (robot description, xacro)
@@ -1,10 +1,34 @@
 <?xml version="1.0"?>
 <robot name="vehicle" xmlns:xacro="http://www.ros.org/wiki/xacro">
-    <xacro:include filename="$(find sim_vehicle)/urdf/physics.urdf.xacro" />
     <xacro:include filename="$(find sim_vehicle)/sensors/sensors.urdf.xacro" />
     <!-- ***************** -->
     <!--  VEHICLE PHYSICS  -->
     <!-- ***************** -->
-    <xacro:vehicle_physics name="vehicle"/>
+    <!-- BASE_LINK -->
+    <link name="base_link">
+        <inertial>
+            <mass value="10.0" />
+            <origin xyz="0 0 0" />
+            <inertia ixx="1" ixy="0" ixz="0.0" iyy="1" iyz="0.0" izz="1" />
+        </inertial>
+        <visual>
+            <origin xyz="0 0 0" rpy="0 0 0" />
+            <geometry>
+                <mesh filename="package://sim_vehicle/meshes/vehicle.dae" />
+            </geometry>
+        </visual>
+        <collision>
+            <origin xyz="0 0 0.5" rpy="0 0 0" />
+            <geometry>
+                <box size="1 1 1" />
+            </geometry>
+        </collision>
+        <gazebo>
+            <plugin filename="libmodel2gazebo.so" name="model2gazebo">
+                <node_name>model2gazebo</node_name>
+                <rate>100</rate>
+            </plugin>
+        </gazebo>
+    </link>
     <!-- *************** -->
     <!--  MAIN SENSORS   -->
