Commit message: simulation corrections

File: sim_vehicle/sensors/camera.urdf.xacro (robot description, xacro)
@@ -15,5 +15,4 @@
                 <box size="${camera_link} ${camera_link} ${camera_link}" />
             </geometry>
-            <material name="red" />
         </visual>
         <inertial>

File: sim_vehicle/sensors/sensors.urdf.xacro (robot description, xacro)
@@ -2,14 +2,5 @@
 <robot xmlns:xacro="http://www.ros.org/wiki/xacro">
     <!-- IMU (Inertal Motion Unit) -->
-    <gazebo>
-        <plugin name="imu_plugin" filename="libgazebo_ros_imu.so">
-            <alwaysOn>true</alwaysOn>
-            <bodyName>base_link</bodyName>
-            <topicName>imu</topicName>
-            <serviceName>imu_service</serviceName>
-            <gaussianNoise>0.0</gaussianNoise>
-            <updateRate>20.0</updateRate>
-        </plugin>
-    </gazebo>
+    <xacro:include filename="$(find sim_vehicle)/sensors/imu.urdf.xacro"/>
     <!-- Camera Front -->
     <xacro:include filename="$(find sim_vehicle)/sensors/camera.urdf.xacro"/>

File: sim_vehicle/urdf/vehicle.urdf.xacro (robot description, xacro)
@@ -16,5 +16,5 @@
         </inertial>
         <visual>
-            <origin xyz="0 0 0" rpy="0 0 1.57" />
+            <origin xyz="0 0 0" rpy="0 0 -1.57" />
             <geometry>
                 <mesh filename="package://sim_vehicle/meshes/drone.dae" />

Commit message: simulation improvements | Works with PID

File: sim_vehicle/sensors/camera.urdf.xacro (robot description, xacro)
@@ -24,5 +24,5 @@
     <joint name="camera_joint" type="fixed">
         <axis xyz="0 0 0" />
-        <origin xyz="0 0 0" rpy="0 0 0" />
+        <origin xyz="0.08 0 0" rpy="0 0 0" />
         <parent link="base_link" />
         <child link="camera_link" />
@@ -58,5 +58,5 @@
                 <imageTopicName>image_raw</imageTopicName>
                 <cameraInfoTopicName>camera_info</cameraInfoTopicName>
-                <frameName>camera_link</frameName>
+                <frameName>base_link</frameName>
                 <hackBaseline>0.07</hackBaseline>
                 <distortionK1>0.0</distortionK1>
