Commit message: parameters load correctly

File: sim_vehicle/urdf/vehicle.urdf.xacro (robot description, xacro)
@@ -13,7 +13,7 @@
             <mass value="${params['mass']}" />
             <origin xyz="0 0 0" />
-            <inertia ixx="${params['inertial']['ixx']}" ixy="${params['inertial']['ixy']}" ixz="${params['inertial']['ixz']}"
-                     iyx="${params['inertial']['iyx']}" iyy="${params['inertial']['iyy']}" iyz="${params['inertial']['iyz']}"
-                     izx="${params['inertial']['izx']}" izy="${params['inertial']['izy']}" izz="${params['inertial']['izz']}"/>
+            <inertia ixx="${params['inertial']['xx']}" ixy="${params['inertial']['xy']}" ixz="${params['inertial']['xz']}"
+                     iyy="${params['inertial']['yy']}" iyz="${params['inertial']['yz']}"
+                     izz="${params['inertial']['zz']}"/>
         </inertial>
         <visual>
@@ -24,7 +24,7 @@
         </visual>
         <collision>
-            <origin xyz="0 0.5 0" rpy="0 0 0" />
+            <origin xyz="0 0 0" rpy="0 0 0" />
             <geometry>
-                <box size="1 1 1" />
+                <sphere radius="0.3"/>
             </geometry>
         </collision>
@@ -35,4 +35,5 @@
             <node_name>model2gazebo</node_name>
             <rate>100</rate>
+            <yaml_config>$(arg params)</yaml_config>
         </plugin>
     </gazebo>

Commit message: drone model preparation

File: sim_vehicle/urdf/vehicle.urdf.xacro (robot description, xacro)
@@ -20,5 +20,5 @@
             <origin xyz="0 0 0" rpy="0 0 0" />
             <geometry>
-                <mesh filename="package://sim_vehicle/meshes/vehicle.dae" />
+                <mesh filename="package://sim_vehicle/meshes/drone.dae" />
             </geometry>
         </visual>
@@ -26,5 +26,5 @@
             <origin xyz="0 0 0" rpy="0 0 0" />
             <geometry>
-                <sphere radius="0.3"/>
+                <sphere radius="0.075"/>
             </geometry>
         </collision>

Commit message: visualization improved

File: sim_vehicle/urdf/vehicle.urdf.xacro (robot description, xacro)
@@ -16,5 +16,5 @@
         </inertial>
         <visual>
-            <origin xyz="0 0 0" rpy="0 0 0" />
+            <origin xyz="0 0 0" rpy="0 0 1.57" />
             <geometry>
                 <mesh filename="package://sim_vehicle/meshes/drone.dae" />
