Commit message: car model applied

File: sim_vehicle/urdf/vehicle_car.urdf.xacro (robot description, xacro)
@@ -16,5 +16,5 @@
         </inertial>
         <visual>
-            <origin xyz="0 0 0" rpy="0 0 -1.57" />
+            <origin xyz="0 0 0" rpy="0 0 0" />
             <geometry>
                 <mesh filename="package://sim_vehicle/meshes/vehicle.dae" />

Commit message: works

File: sim_vehicle/urdf/vehicle_car.urdf.xacro (robot description, xacro)
@@ -22,5 +22,5 @@
         </visual>
         <collision>
-            <origin xyz="0 0 0" rpy="0 0 0" />
+            <origin xyz="0 0 ${params['height'] / 2}" rpy="0 0 0" />
             <geometry>
                 <!-- <sphere radius="0.075"/> -->
